Commit message: adding_gripper

File: tb4_simulation/ur5e_cartesian_control/urdf/gripper.xacro (robot description, xacro)
@@ -1,8 +1,19 @@
-<robot xmlns:xacro="http://ros.org/wiki/xacro" name="robotiq_85_gripper">
-  <xacro:include filename="$(find ur5e_cartesian_control)/urdf/robotiq_85_gripper.urdf.xacro" />
-  <xacro:macro name="add_gripper" params="parent">
-    <xacro:robotiq_85_gripper prefix="" parent="${parent}">
-      <origin xyz="0 0 0" rpy="0 -1.57 0"/>
-    </xacro:robotiq_85_gripper>
+<?xml version="1.0"?>
+<robot xmlns:xacro="http://www.ros.org/wiki/xacro">
+  <xacro:include filename="$(find robotiq_description)/urdf/ur_to_robotiq_adapter.urdf.xacro"/>
+  <xacro:include filename="$(find robotiq_description)/urdf/robotiq_2f_85_macro.urdf.xacro"/>
+  <xacro:macro name="add_gripper" params="parent:=tool0 prefix:=rq_ sim_ignition:=false use_fake_hardware:=false">
+    <xacro:ur_to_robotiq
+        connected_to="${parent}"
+        prefix="${prefix}" />
+  <xacro:robotiq_gripper
+        name="robotiq_85"
+        parent="${prefix}ur_to_robotiq_link"
+        prefix="${prefix}"
+        sim_ignition="${sim_ignition}"
+        use_fake_hardware="${use_fake_hardware}"
+        include_ros2_control="true">
+  <origin xyz="0 0 0" rpy="0 0 0"/>
+</xacro:robotiq_gripper>
   </xacro:macro>
 </robot>

File: tb4_simulation/ur5e_cartesian_control/urdf/ur5e_cartesian.urdf.xacro (robot description, xacro)
@@ -6,5 +6,5 @@
   <xacro:include filename="$(find ur_description)/urdf/ur_macro.xacro" />
   <xacro:include filename="$(find se3_sensor_driver)/urdf/se3_sensor.xacro"/>
-  <!-- <xacro:include filename="$(find ur5e_cartesian_control)/urdf/gripper.xacro" /> -->
+  <xacro:include filename="$(find ur5e_cartesian_control)/urdf/gripper.xacro" />
   <xacro:arg name="joint_limit_params" default="$(find ur_description)/config/$(arg ur_type)/joint_limits.yaml"/>
   <xacro:arg name="kinematics_params" default="$(find ur_description)/config/$(arg ur_type)/default_kinematics.yaml"/>
@@ -28,5 +28,8 @@
     <origin xyz="0 0 0" rpy="0 0 0" />
   </xacro:ur_robot>
-  <!-- <xacro:add_gripper parent="tool0" /> -->
+  <xacro:add_gripper parent="tool0"
+                   prefix="rq_"
+                   sim_ignition="$(arg sim_ignition)"
+                   use_fake_hardware="$(arg use_fake_hardware)"/>
   <gazebo>
     <plugin filename="libign_ros2_control-system.so" name="ign_ros2_control::IgnitionROS2ControlPlugin">
